File: hw/design/controller_ild8150/controller.kicad_pcb (KiCad board)
At the start: 2 copper layers, 35 x 21.7 mm, 45 parts, among them J1 Conn_ARM_SWD_TagConnect_TC203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, J3 Conn_02x01, U1 ATSAMC21E18A-MNT, U3 ILD8150, U4 MCP2021A-330E/SN

Commit message: Hardware schematic cleanup
Parts:
- renumbered C13 to C300, C14 to C301, C12 to C302, C15 to C303, C9 to C400, C6 to C401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
