File: hw/design/controller_tld509x/controller.kicad_pcb (KiCad board)
At the start: 4 copper layers, 35 x 21.7 mm, 53 parts, among them J1 Conn_ARM_SWD_TagConnect_TC203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, J3 Conn_02x01, Q1 PSMN5R2-60YL, Q3 2N7002, Q5 SiSS27DN, U1 ATSAMC21E18A-MNT, U2 TLD509x, U4 MCP2021A-330E/SN

Commit message: Final hardware design
Changed lines of the file:
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@@
       (outputformat 1)
       (mirror false)
-      (drillshape 1)
+      (drillshape 0)
       (scaleselection 1)
-      (outputdirectory "")
+      (outputdirectory "../../../../ordering-2024-05/controller-tld509x/")
     )
   )
@@
     (fp_line (start 1.6 0.8) (end -1.6 0.8)
       (stroke (width 0.1) (type solid)) (layer "F.Fab"))
-    (pad "1" smd roundrect (at -1.4625 0) (size 1.125 1.75) (layers "F.Cu" "F.Paste" "F.Mask") (roundrect_rratio 0.222222)
+    (pad "1" smd roundrect (at -1.4625 0) (size 1.125 1.75) (layers "F.Cu" "F.Paste" "F.Mask") (roundrect_rratio 0.2222222222)
       (net 47 "/TLD509x_FB_P") (pintype "passive"))
-    (pad "2" smd roundrect (at 1.4625 0) (size 1.125 1.75) (layers "F.Cu" "F.Paste" "F.Mask") (roundrect_rratio 0.222222)
+    (pad "2" smd roundrect (at 1.4625 0) (size 1.125 1.75) (layers "F.Cu" "F.Paste" "F.Mask") (roundrect_rratio 0.2222222222)
       (net 46 "/TLD509x_FB_N") (pintype "passive"))
     (model "${KICAD6_3DMODEL_DIR}/Resistor_SMD.3dshapes/R_1206_3216Metric.wrl"
@@
     (fp_line (start 2.5 2.5) (end -2.5 2.5)
       (stroke (width 0.1) (type solid)) (layer "F.Fab"))
-    (pad "" smd roundrect (at -0.875 -0.875 180) (size 1.41 1.41) (layers "F.Paste") (roundrect_rratio 0.177305))
-    (pad "" smd roundrect (at -0.875 0.875 180) (size 1.41 1.41) (layers "F.Paste") (roundrect_rratio 0.177305))
-    (pad "" smd roundrect (at 0.875 -0.875 180) (size 1.41 1.41) (layers "F.Paste") (roundrect_rratio 0.177305))
-    (pad "" smd roundrect (at 0.875 0.875 180) (size 1.41 1.41) (layers "F.Paste") (roundrect_rratio 0.177305))
+    (pad "" smd roundrect (at -0.875 -0.875 180) (size 1.41 1.41) (layers "F.Paste") (roundrect_rratio 0.1773049645))
+    (pad "" smd roundrect (at -0.875 0.875 180) (size 1.41 1.41) (layers "F.Paste") (roundrect_rratio 0.1773049645))
+    (pad "" smd roundrect (at 0.875 -0.875 180) (size 1.41 1.41) (layers "F.Paste") (roundrect_rratio 0.1773049645))
+    (pad "" smd roundrect (at 0.875 0.875 180) (size 1.41 1.41) (layers "F.Paste") (roundrect_rratio 0.1773049645))
     (pad "1" smd roundrect (at -2.45 -1.75 180) (size 0.8 0.25) (layers "F.Cu" "F.Paste" "F.Mask") (roundrect_rratio 0.25)
       (net 49 "unconnected-(U1-PA00-Pad1)") (pinfunction "PA00") (pintype "bidirectional+no_connect"))
@@
     (fp_line (start 1 0.625) (end 1 -0.625)
       (stroke (width 0.1) (type solid)) (layer "B.Fab"))
-    (pad "1" smd roundrect (at -0.9125 0 270) (size 1.025 1.4) (layers "B.Cu" "B.Paste" "B.Mask") (roundrect_rratio 0.243902)
+    (pad "1" smd roundrect (at -0.9125 0 270) (size 1.025 1.4) (layers "B.Cu" "B.Paste" "B.Mask") (roundrect_rratio 0.243902439)
       (net 1 "GND") (pintype "passive") (zone_connect 2))
-    (pad "2" smd roundrect (at 0.9125 0 270) (size 1.025 1.4) (layers "B.Cu" "B.Paste" "B.Mask") (roundrect_rratio 0.243902)
+    (pad "2" smd roundrect (at 0.9125 0 270) (size 1.025 1.4) (layers "B.Cu" "B.Paste" "B.Mask") (roundrect_rratio 0.243902439)
       (net 42 "/TLD509x_CS") (pintype "passive"))
     (model "${KICAD6_3DMODEL_DIR}/Resistor_SMD.3dshapes/R_0805_2012Metric.wrl"

Commit message: Hardware schematic cleanup
Parts:
- C404: renamed from C4; value 220n -> 100n
- C502: renamed from C21; value 4.7u -> 10u
- C504: renamed from C20; value 220n -> 100n
- C505: renamed from C19; value 47n -> 22n
- C506: renamed from C22; value 47n -> 100n
- Q500: renamed from Q5; value SiSS27DN -> BUK6Y24-40PX
- Q501: renamed from Q1; value PSMN5R2-60YL -> BUK7Y7R0-40HX
- R506: renamed from R8; value 20k -> 4.7k
- U300: renamed from U4; value MCP2021A-330E/SN -> MCP2021A-500E/SN
- renumbered C13 to C300, C14 to C301, C12 to C302, C15 to C303, C9 to C400, C6 to C401, C7 to C402, C1 to C403, C8 to C405, C17 to C500, C2 to C501, C18 to C503, D8 to D200, D3 to D300, D7 to D500, D6 to D501, D5 to D502, D1 to D503, J1 to J400, J3 to J500, L1 to L400, L2 to L500, Q3 to Q502, R5 to R300, R4 to R301, R1 to R400, R2 to R401, R3 to R402, R15 to R500, R17 to R501, R14 to R502, R10 to R503, R11 to R504, R9 to R505, R6 to R507, R16 to R508, R12 to R509, R13 to R510, TH1 to TH400, U5 to U100, U1 to U400, U2 to U500
