File: hw/design/controller_al8891/controller.kicad_pcb (KiCad board)
At the start: 4 copper layers, 35 x 21.7 mm, 64 parts, among them J1 Conn_02x01, J501 Conn_ARM_SWD_TagConnect_TC203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, Q200 SIA469DJ-T1-GE3, U1 TPS629210DRLR, U300 MCP2003BT-E/MC, U500 ATSAMD21E18A-MUT, U800 AL8891

Commit message: Finalized design (JLC ordered)
Parts:
- C808: value 2.2u -> 1u
- R805: value 290m -> 300m
- R820: value 237k -> 200k
- R823: value 10k -> 120k
- R824: value 10k -> 27k
- R825: value 10k -> 1k
- renumbered C1 to C401, C2 to C403, C5 to C504, C3 to C506, C4 to C507, C6 to C508, C7 to C807, J1 to J811, R1 to R305, U1 to U400
Connections:
- net M07_VMON renamed M09_VMON
