File: hw/design/controller_al8891/controller.kicad_sch (KiCad schematic)
At the start: 66 parts, among them J1 Conn_02x01, J501 Conn_ARM_SWD_TagConnect_TC203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, Q200 SIA469DJ-T1-GE3, U1 TPS629210DRLR, U300 MCP2003BT-E/MC, U500 ATSAMD21E18A-MUT, U800 AL8891

Commit message: Finalized design (JLC ordered)
Parts:
- removed FID1, FID2: Fiducial, symbol Mechanical:Fiducial
- C807: renamed from C7; now not fitted
- C808: value 2.2u -> 1u
- C826: now not fitted
- R305: renamed from R1; now not fitted
- R805: value 290m -> 300m
- R815: now fitted
- R820: value 237k -> 200k
- R823: value 10k -> 120k
- R824: value 10k -> 27k
- R825: value 10k -> 1k
- renumbered C1 to C401, C2 to C403, C5 to C504, C3 to C506, C4 to C507, C6 to C508, J1 to J811, U1 to U400
Connections:
- net M07_VMON renamed M09_VMON
- no-connect marks 3 -> 16
Other:
- note added: "Mechanical"
- note added: "Place NTC close to LED"
- note added: "clearance!"
- note added: "fSW ~500kHz"
- note added: "keep C401 close to VIN of U400"
- note added: "keep C504,C505 close to VDDANA pin of U500"
- note added: "keep C506,C507 close to VDDIN pin of U500"
- note added: "keep C508 close to VDDCORE pin of U500"
- note added: "keep C801,C802,C827 close to VIN pin of U800 keep C808 close to VCC pin of U800 put C803 across CBOOT/SW pin of U800"
- note added: "return path shall be clear"
- note added: "route close, guard vias"
- note removed: "3.3V / 24.7k = 133uA"
- note removed: "AIN 1"
- note removed: "AIN 2"
- note removed: "AIN19"
- note removed: "DAC VOUT"
- note removed: "EXTINT6"
- note removed: "EXTINT7"
- note removed: "GPIO"
- note removed: "Keep close, guard vias"
- note removed: "Place NTC behind LED"
- note removed: "SERCOM1 PAD0"
- note removed: "SERCOM1 PAD1"
- note removed: "TCC0 W0"
- note removed: "TODO: cap sizes"
- note removed: "TODO: cap value"
- note removed: "TODO: output capacitance?"
- note removed: "TODO: resistor value"
- note removed: "VCCQ=5V@30mA"
- note removed: "keep C10,C12 close to VDDIN pin of U6"
- note removed: "keep C13,C15 close to VDDANA pin of U6"
- note removed: "keep C17 close to VDDCORE pin of U6"
- moved on the sheet: C301, C302, C304, C401, C403, C504, C505, C506, C507, C508, C510, C801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
